File: src/Moirai.kicad_sch (KiCad schematic)
At the start: 36 parts, among them J1 Screw_Terminal_01x02, Q1 BS170, Q2 BS170, Q3 BS170, Q4 BC850, U1 74LS279, U2 74HC00, U3 74HC00, U4 AMS1117-5.0

Commit message: updated schematic
Parts:
- added J2: Screw_Terminal_01x02, symbol Connector:Screw_Terminal_01x02
- added Q5: IPP80P03P4L-04, symbol IPP80P03P4L:IPP80P03P4L-04
- added R14: 10kR, symbol Device:R_Small
Connections:
- net GND: now also Q4.2 (E), J2.2 (Pin_2)
- net OUT: now also Q4.1 (B)
- net VCC: now also Q5.P3, R14.1
- net at Q4.3 (C): now also Q5.P1, R14.2
- new net: J2.1 (Pin_1), Q5.P2
Other:
- moved on the sheet: C1, C4, C7, C8, D3, J1, JP3, Q3, Q4, R10, R11, R7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

Commit message: updated schematic
Parts:
- added J3: Screw_Terminal_01x06, TerminalBlock_WAGO:TerminalBlock_WAGO_236-406_1x06_P5.00mm_45Degree, symbol Connector:Screw_Terminal_01x06
- C1, C5, C6, C7, C8: footprint (none) -> Capacitor_SMD:C_0805_2012Metric
- C2, C3, C4: value C_Small -> 1uF; footprint (none) -> Capacitor_SMD:C_0805_2012Metric
- D1, D2, D3: footprint (none) -> Diode_SMD:D_SMA
- J1, J2: footprint (none) -> TerminalBlock_WAGO:TerminalBlock_WAGO_236-402_1x02_P5.00mm_45Degree
- Q5: footprint (none) -> Package_TO_SOT_THT:TO-220-3_Vertical
- R1, R10, R11, R12, R13, R14, R2, R3, R4, R5, R6, R7, R8, R9: footprint (none) -> Resistor_SMD:R_0805_2012Metric
- U1: footprint (none) -> Package_DIP:DIP-16_W7.62mm
- U2, U3: footprint (none) -> Package_DIP:DIP-14_W7.62mm
Connections:
- net CH1_CONN: now also J3.1 (Pin_1)
- net CH2_CONN: now also J3.3 (Pin_3)
- net CH3_CONN: now also J3.5 (Pin_5)
- net GND: now also J3.2 (Pin_2), J3.4 (Pin_4), J3.6 (Pin_6)
Other:
- note removed: "A 2S (7.4V) battery should be used"

Commit message: fixed IPP80P symbol
Connections:
- net VCC: now also Q5.3; no longer Q5.P3
- net at Q4.3 (C), R14.2: now also Q5.1; no longer Q5.P1
- net at J2.1 (Pin_1): now also Q5.2; no longer Q5.P2
Changed lines of the file:
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@@
 			)
 		)
-		(pin "P2"
+		(pin "3"
 		)
-		(pin "P1"
+		(pin "1"
 		)
-		(pin "P3"
+		(pin "2"
 		)
 		(instances

Commit message: PCB design
Parts:
- removed J1: Screw_Terminal_01x02, TerminalBlock_WAGO:TerminalBlock_WAGO_236-402_1x02_P5.00mm_45Degree, symbol Connector:Screw_Terminal_01x02
- added J1: Conn_01x02, Connector_AMASS:AMASS_XT30U-M_1x02_P5.0mm_Vertical, symbol Connector_Generic:Conn_01x02
Connections:
- net GND: now also J1.1 (Pin_1)
- net VCC: now also J1.2 (Pin_2)
Changed lines of the file:
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@@
 	(wire
 		(pts
-			(xy 137.16 179.07) (xy 137.16 176.53)
-		)
-		(stroke
-			(width 0)
-			(type default)
-		)
-	)
-	(wire
-		(pts
 			(xy 73.66 38.1) (xy 87.63 38.1)
 		)
@@
 	(wire
 		(pts
-			(xy 210.82 142.24) (xy 210.82 143.51)
+			(xy 137.16 179.07) (xy 137.16 176.53)
 		)
 		(stroke
@@
 	(wire
 		(pts
-			(xy 198.12 101.6) (xy 200.66 101.6)
+			(xy 210.82 142.24) (xy 210.82 143.51)
 		)
 		(stroke
@@
 	(wire
 		(pts
-			(xy 30.48 55.88) (xy 30.48 59.69)
+			(xy 198.12 101.6) (xy 200.66 101.6)
 		)
 		(stroke
@@
 	(wire
 		(pts
-			(xy 139.7 179.07) (xy 137.16 179.07)
+			(xy 30.48 55.88) (xy 30.48 59.69)
 		)
 		(stroke
@@
 	(wire
 		(pts
-			(xy 139.7 181.61) (xy 137.16 181.61)
-		)
-		(stroke
-			(width 0)
-			(type default)
-		)
-	)
-	(wire
-		(pts
 			(xy 53.34 87.63) (xy 53.34 92.71)
 		)
@@
 	(wire
 		(pts
-			(xy 137.16 181.61) (xy 137.16 184.15)
+			(xy 137.16 184.15) (xy 137.16 181.61)
 		)
 		(stroke
@@
 	(wire
 		(pts
+			(xy 139.7 179.07) (xy 137.16 179.07)
+		)
+		(stroke
+			(width 0)
+			(type default)
+		)
+	)
+	(wire
+		(pts
 			(xy 210.82 154.94) (xy 210.82 157.48)
 		)
@@
 	(wire
 		(pts
+			(xy 137.16 181.61) (xy 139.7 181.61)
+		)
+		(stroke
+			(width 0)
+			(type default)
+		)
+	)
+	(wire
+		(pts
 			(xy 53.34 121.92) (xy 41.91 121.92)
 		)
@@
 	)
 	(symbol
-		(lib_id "Connector:Screw_Terminal_01x02")
-		(at 144.78 179.07 0)
+		(lib_id "Connector_Generic:Conn_01x02")
+		(at 144.78 181.61 0)
+		(mirror x)
 		(unit 1)
 		(exclude_from_sim no)
@@
 		(on_board yes)
 		(dnp no)
-		(fields_autoplaced yes)
 		(property "Reference" "J1"
-			(at 147.32 179.0699 0)
+			(at 147.32 181.6101 0)
 			(effects
 				(font
@@
 			)
 		)
-		(property "Value" "Screw_Terminal_01x02"
-			(at 147.32 181.6099 0)
+		(property "Value" "Conn_01x02"
+			(at 147.32 179.0701 0)
 			(effects
 				(font
@@
 			)
 		)
-		(property "Footprint" "TerminalBlock_WAGO:TerminalBlock_WAGO_236-402_1x02_P5.00mm_45Degree"
-			(at 144.78 179.07 0)
+		(property "Footprint" "Connector_AMASS:AMASS_XT30U-M_1x02_P5.0mm_Vertical"
+			(at 144.78 181.61 0)
 			(effects
 				(font
@@
 		)
 		(property "Datasheet" "~"
-			(at 144.78 179.07 0)
+			(at 144.78 181.61 0)
 			(effects
 				(font
@@
 			)
 		)
-		(property "Description" "Generic screw terminal, single row, 01x02, script generated (kicad-library-utils/schlib/autogen/connector/)"
-			(at 144.78 179.07 0)
+		(property "Description" "Generic connector, single row, 01x02, script generated (kicad-library-utils/schlib/autogen/connector/)"
+			(at 144.78 181.61 0)
 			(effects
 				(font
