File: src/Moirai.kicad_pcb (KiCad board)
At the start: 2 copper layers, 50 parts, among them J1 Conn_01x02, J2 Screw_Terminal_01x02, J3 Screw_Terminal_01x06, Q1 BS170, Q2 BS170, Q3 BS170, Q4 BC850, Q5 IPP80P03P4L-04, U1 74LS279, U2 74HC00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

Commit message: PCB update
Parts:
- moved REF** 191.2 mm to (228.6, 62.5)
- moved REF** 191.0 mm to (228.6, 103.5)
- moved Q5 179.9 mm to (227.3, 21.9), turned to -90 degrees
- moved R14 179.3 mm to (223.1, 26.0), turned to 90 degrees
- moved Q4 173.9 mm to (223.1, 21.4), turned to -90 degrees
- moved J2 173.4 mm to (235.2, 24.4)
- moved U3 143.0 mm to (179.9, 26.4)
- moved U2 142.6 mm to (168.7, 26.4)
- moved C6 140.7 mm to (183.8, 22.2), turned to 180 degrees
- moved C7 137.9 mm to (203.2, 18.8)
- moved R12 137.7 mm to (190.7, 31.4), turned to 180 degrees
- moved R9 136.3 mm to (150.1, 34.5), turned to 180 degrees
- moved R13 136.1 mm to (190.7, 28.8), turned to 180 degrees
- moved JP1 133.9 mm to (266.7, 31.5)
- moved JP2 133.9 mm to (266.7, 36.0)
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